Commit message: Loading Working.

File: resource/Nomad/Nomad_leg_test.urdf (robot description, URDF)
Before this commit: robot Nomad, 6 links, 5 joints
Links:
- added link world
Joints:
- added joint leg_to_world_fixed: type fixed, parent world, child base_link, origin xyz=0 0.0 0.5 rpy=0 0 0

Commit message: More DART experimenting

File: resource/Nomad/Nomad_leg_test.urdf (robot description, URDF)
Before this commit: robot Nomad, 7 links, 6 joints
Links:
- removed link Foot1
- removed link HFE_Actuator1
- removed link KFE_Actuator1
- removed link Lower_Leg1
- removed link Upper_Leg1
- added link Foot, mass 0.07686399002843462; collision mesh filename=meshes/Foot1.stl scale=0.001 0.001 0.001; visual mesh filename=meshes/Foot1.stl scale=0.001 0.001 0.001
- added link HFE_Actuator, mass 0.22819661408568134; collision mesh filename=meshes/HFE_Actuator1.stl scale=0.001 0.001 0.001; visual mesh filename=meshes/HFE_Actuator1.stl scale=0.001 0.001 0.001
- added link KFE_Actuator, mass 0.3024397808873297; collision mesh filename=meshes/KFE_Actuator1.stl scale=0.001 0.001 0.001; visual mesh filename=meshes/KFE_Actuator1.stl scale=0.001 0.001 0.001
- added link Lower_Leg, mass 0.1002751137848322; collision mesh filename=meshes/Lower_Leg1.stl scale=0.001 0.001 0.001; visual mesh filename=meshes/Lower_Leg1.stl scale=0.001 0.001 0.001
- added link Upper_Leg, mass 0.28719650282800196; collision mesh filename=meshes/Upper_Leg1.stl scale=0.001 0.001 0.001; visual mesh filename=meshes/Upper_Leg1.stl scale=0.001 0.001 0.001
Joints:
- joint base_to_hip_motor: child HFE_Actuator1 -> HFE_Actuator
- joint hip_motor_to_knee_motor: child KFE_Actuator1 -> KFE_Actuator; parent HFE_Actuator1 -> HFE_Actuator
- joint knee_motor_upper_leg: child Upper_Leg1 -> Upper_Leg; parent KFE_Actuator1 -> KFE_Actuator
- joint knee_to_foot: child Foot1 -> Foot; parent Lower_Leg1 -> Lower_Leg
- joint upper_leg_to_lower_leg: child Lower_Leg1 -> Lower_Leg; parent Upper_Leg1 -> Upper_Leg

Commit message: Ready for PD test

File: resource/Nomad/Nomad_leg_test.urdf (robot description, URDF)
Before this commit: robot Nomad, 7 links, 6 joints
Links:
- removed link Foot
- removed link HFE_Actuator
- removed link KFE_Actuator
- removed link Lower_Leg
- removed link Upper_Leg
- added link foot, mass 0.07686399002843462; collision mesh filename=meshes/Foot1.stl scale=0.001 0.001 0.001; visual mesh filename=meshes/Foot1.stl scale=0.001 0.001 0.001
- added link hfe_motor, mass 0.22819661408568134; collision mesh filename=meshes/HFE_Actuator1.stl scale=0.001 0.001 0.001; visual mesh filename=meshes/HFE_Actuator1.stl scale=0.001 0.001 0.001
- added link kfe_motor, mass 0.3024397808873297; collision mesh filename=meshes/KFE_Actuator1.stl scale=0.001 0.001 0.001; visual mesh filename=meshes/KFE_Actuator1.stl scale=0.001 0.001 0.001
- added link lower_Leg, mass 0.1002751137848322; collision mesh filename=meshes/Lower_Leg1.stl scale=0.001 0.001 0.001; visual mesh filename=meshes/Lower_Leg1.stl scale=0.001 0.001 0.001
- added link upper_Leg, mass 0.28719650282800196; collision mesh filename=meshes/Upper_Leg1.stl scale=0.001 0.001 0.001; visual mesh filename=meshes/Upper_Leg1.stl scale=0.001 0.001 0.001
Joints:
- removed joint base_to_hip_motor
- removed joint hip_motor_to_knee_motor
- removed joint leg_to_world_fixed
- removed joint upper_leg_to_lower_leg
- added joint base_to_hfe_motor: type fixed, parent base_link, child hfe_motor, origin xyz=0.013417 -0.051438 -0.030983 rpy=0 0 0
- added joint hfe_motor_to_kfe_motor: type continuous, parent hfe_motor, child kfe_motor, origin xyz=0.0 -0.047 0.0 rpy=0 0 0, axis 0.0 -1.0 -0.0
- added joint kfe_joint: type continuous, parent upper_Leg, child lower_Leg, origin xyz=2e-06 -0.018 -0.25 rpy=0 0 0, axis 0.0 -1.0 -0.0
- added joint leg_to_world: type prismatic, parent world, child base_link, origin xyz=0 0.0 0.0 rpy=0 0 0, axis 0.0 0.0 1.0, limit lower=-1.0 upper=3.0 effort=1000.0 velocity=100.0
- joint knee_motor_upper_leg: child Upper_Leg -> upper_Leg; parent KFE_Actuator -> kfe_motor
- joint knee_to_foot: child Foot -> foot; parent Lower_Leg -> lower_Leg

Commit message: Add Input Handling/Target

File: resource/Nomad/Nomad_leg_test.urdf (robot description, URDF)
Before this commit: robot Nomad, 7 links, 6 joints
Joints:
- removed joint hfe_motor_to_kfe_motor
- added joint hfe_joint: type continuous, parent hfe_motor, child kfe_motor, origin xyz=0.0 -0.047 0.0 rpy=0 0 0, axis 0.0 -1.0 -0.0

Commit message: Add PD Controller, and External Force Test.

File: resource/Nomad/Nomad_leg_test.urdf (robot description, URDF)
Before this commit: robot Nomad, 7 links, 6 joints
Links:
- link base_link: mass 7.166707013041554 -> 4.166707013041554

Commit message: Add Feed Forward Gravity

File: resource/Nomad/Nomad_leg_test.urdf (robot description, URDF)
Before this commit: robot Nomad, 7 links, 6 joints
Links:
- link base_link: mass 4.166707013041554 -> 7.166707013041554
