Commit message: Update URDF

File: resource/NomadFull/Nomad.urdf (robot description, URDF)
Before this commit: robot Nomad, 25 links, 24 joints
Links:
- removed link foot_FL1
- removed link foot_FR1
- removed link foot_RL1
- removed link foot_RR1
- removed link haa_FL_link1
- removed link haa_FR_link1
- removed link haa_RL_link1
- removed link haa_RR_link1
- removed link hfe_FL_link1
- removed link hfe_FR_link1
- removed link hfe_RL_link1
- removed link hfe_RR_link1
- removed link kfe_FL_link1
- removed link kfe_FR_link1
- removed link kfe_RL_link1
- removed link kfe_RR_link1
- removed link lower_leg_FL_link1
- removed link lower_leg_FR_link1
- removed link lower_leg_RL_link1
- removed link lower_leg_RR_link1
- removed link upper_leg_FL_link1
- removed link upper_leg_FR_link1
- removed link upper_leg_RL_link1
- removed link upper_leg_RR_link1
- added link b_foot_FL, mass 0.07686399002843429; collision mesh filename=meshes/b_foot_FL.stl scale=0.001 0.001 0.001; visual mesh filename=meshes/b_foot_FL.stl scale=0.001 0.001 0.001
- added link b_foot_FR, mass 0.07686399002843429; collision mesh filename=meshes/b_foot_FR.stl scale=0.001 0.001 0.001; visual mesh filename=meshes/b_foot_FR.stl scale=0.001 0.001 0.001
- added link b_foot_RL, mass 0.07686399002843429; collision mesh filename=meshes/b_foot_RL.stl scale=0.001 0.001 0.001; visual mesh filename=meshes/b_foot_RL.stl scale=0.001 0.001 0.001
- added link b_foot_RR, mass 0.07686399002843429; collision mesh filename=meshes/b_foot_RR.stl scale=0.001 0.001 0.001; visual mesh filename=meshes/b_foot_RR.stl scale=0.001 0.001 0.001
- added link b_haa_motor_FL, mass 0.22819661408568134; collision mesh filename=meshes/b_haa_motor_FL.stl scale=0.001 0.001 0.001; visual mesh filename=meshes/b_haa_motor_FL.stl scale=0.001 0.001 0.001
- added link b_haa_motor_FR, mass 0.22819661408568134; collision mesh filename=meshes/b_haa_motor_FR.stl scale=0.001 0.001 0.001; visual mesh filename=meshes/b_haa_motor_FR.stl scale=0.001 0.001 0.001
- added link b_haa_motor_RL, mass 0.22819661408568134; collision mesh filename=meshes/b_haa_motor_RL.stl scale=0.001 0.001 0.001; visual mesh filename=meshes/b_haa_motor_RL.stl scale=0.001 0.001 0.001
- added link b_haa_motor_RR, mass 0.22819661408568134; collision mesh filename=meshes/b_haa_motor_RR.stl scale=0.001 0.001 0.001; visual mesh filename=meshes/b_haa_motor_RR.stl scale=0.001 0.001 0.001
- added link b_hfe_motor_FL, mass 0.2875872093499024; collision mesh filename=meshes/b_hfe_motor_FL.stl scale=0.001 0.001 0.001; visual mesh filename=meshes/b_hfe_motor_FL.stl scale=0.001 0.001 0.001
- added link b_hfe_motor_FR, mass 0.2875872093499024; collision mesh filename=meshes/b_hfe_motor_FR.stl scale=0.001 0.001 0.001; visual mesh filename=meshes/b_hfe_motor_FR.stl scale=0.001 0.001 0.001
- added link b_hfe_motor_RL, mass 0.2875872093499024; collision mesh filename=meshes/b_hfe_motor_RL.stl scale=0.001 0.001 0.001; visual mesh filename=meshes/b_hfe_motor_RL.stl scale=0.001 0.001 0.001
- added link b_hfe_motor_RR, mass 0.2875872093499024; collision mesh filename=meshes/b_hfe_motor_RR.stl scale=0.001 0.001 0.001; visual mesh filename=meshes/b_hfe_motor_RR.stl scale=0.001 0.001 0.001
- added link b_kfe_motor_FL, mass 0.30243979231772933; collision mesh filename=meshes/b_kfe_motor_FL.stl scale=0.001 0.001 0.001; visual mesh filename=meshes/b_kfe_motor_FL.stl scale=0.001 0.001 0.001
- added link b_kfe_motor_FR, mass 0.30244037793017975; collision mesh filename=meshes/b_kfe_motor_FR.stl scale=0.001 0.001 0.001; visual mesh filename=meshes/b_kfe_motor_FR.stl scale=0.001 0.001 0.001
- added link b_kfe_motor_RL, mass 0.30243979231772933; collision mesh filename=meshes/b_kfe_motor_RL.stl scale=0.001 0.001 0.001; visual mesh filename=meshes/b_kfe_motor_RL.stl scale=0.001 0.001 0.001
- added link b_kfe_motor_RR, mass 0.30244037793017975; collision mesh filename=meshes/b_kfe_motor_RR.stl scale=0.001 0.001 0.001; visual mesh filename=meshes/b_kfe_motor_RR.stl scale=0.001 0.001 0.001
- added link b_lower_leg_FL, mass 0.10027511378483192; collision mesh filename=meshes/b_lower_leg_FL.stl scale=0.001 0.001 0.001; visual mesh filename=meshes/b_lower_leg_FL.stl scale=0.001 0.001 0.001
- added link b_lower_leg_FR, mass 0.10027511378483192; collision mesh filename=meshes/b_lower_leg_FR.stl scale=0.001 0.001 0.001; visual mesh filename=meshes/b_lower_leg_FR.stl scale=0.001 0.001 0.001
- added link b_lower_leg_RL, mass 0.10027511378483192; collision mesh filename=meshes/b_lower_leg_RL.stl scale=0.001 0.001 0.001; visual mesh filename=meshes/b_lower_leg_RL.stl scale=0.001 0.001 0.001
- added link b_lower_leg_RR, mass 0.10027511378483192; collision mesh filename=meshes/b_lower_leg_RR.stl scale=0.001 0.001 0.001; visual mesh filename=meshes/b_lower_leg_RR.stl scale=0.001 0.001 0.001
- added link b_upper_leg_FL, mass 0.28719650938086905; collision mesh filename=meshes/b_upper_leg_FL.stl scale=0.001 0.001 0.001; visual mesh filename=meshes/b_upper_leg_FL.stl scale=0.001 0.001 0.001
- added link b_upper_leg_FR, mass 0.28719862886504943; collision mesh filename=meshes/b_upper_leg_FR.stl scale=0.001 0.001 0.001; visual mesh filename=meshes/b_upper_leg_FR.stl scale=0.001 0.001 0.001
- added link b_upper_leg_RL, mass 0.28719650938086905; collision mesh filename=meshes/b_upper_leg_RL.stl scale=0.001 0.001 0.001; visual mesh filename=meshes/b_upper_leg_RL.stl scale=0.001 0.001 0.001
- added link b_upper_leg_RR, mass 0.28719862886504943; collision mesh filename=meshes/b_upper_leg_RR.stl scale=0.001 0.001 0.001; visual mesh filename=meshes/b_upper_leg_RR.stl scale=0.001 0.001 0.001
Joints:
- removed joint base_link_haa_FL
- removed joint base_link_haa_FR
- removed joint base_link_haa_RL
- removed joint base_link_haa_RR
- removed joint haa_to_hfe_FL
- removed joint haa_to_hfe_FR
- removed joint haa_to_hfe_RL
- removed joint haa_to_hfe_RR
- removed joint hfe_to_kfe_FL
- removed joint hfe_to_kfe_FR
- removed joint hfe_to_kfe_RL
- removed joint hfe_to_kfe_RR
- removed joint hfe_to_upper_leg_FL
- removed joint hfe_to_upper_leg_FR
- removed joint hfe_to_upper_leg_RL
- removed joint hfe_to_upper_leg_RR
- removed joint knee_to_foot_FL
- removed joint knee_to_foot_FR
- removed joint knee_to_foot_RL
- removed joint knee_to_foot_RR
- removed joint upper_leg_to_lower_leg_FL
- removed joint upper_leg_to_lower_leg_FR
- removed joint upper_leg_to_lower_leg_RL
- removed joint upper_leg_to_lower_leg_RR
- added joint j_base_link_haa_FL: type fixed, parent base_link, child b_haa_motor_FL, origin xyz=0.215 0.07 0.0 rpy=0 0 0
- added joint j_base_link_haa_FR: type fixed, parent base_link, child b_haa_motor_FR, origin xyz=0.215 -0.07 0.0 rpy=0 0 0
- added joint j_base_link_haa_RL: type fixed, parent base_link, child b_haa_motor_RL, origin xyz=-0.215 0.07 0.0 rpy=0 0 0
- added joint j_base_link_haa_RR: type fixed, parent base_link, child b_haa_motor_RR, origin xyz=-0.215 -0.07 0.0 rpy=0 0 0
- added joint j_haa_FL: type continuous, parent b_haa_motor_FL, child b_hfe_motor_FL, origin xyz=0.002 0.0 0.0 rpy=0 0 0, axis 1.0 0.0 0.0
- added joint j_haa_FR: type continuous, parent b_haa_motor_FR, child b_hfe_motor_FR, origin xyz=0.002 0.0 0.0 rpy=0 0 0, axis 1.0 0.0 -0.0
- added joint j_haa_RL: type continuous, parent b_haa_motor_RL, child b_hfe_motor_RL, origin xyz=-0.002 0.0 0.0 rpy=0 0 0, axis -1.0 -0.0 -0.0
- added joint j_haa_RR: type continuous, parent b_haa_motor_RR, child b_hfe_motor_RR, origin xyz=-0.002 0.0 0.0 rpy=0 0 0, axis -1.0 -0.0 -0.0
- added joint j_hfe_FL: type continuous, parent b_hfe_motor_FL, child b_kfe_motor_FL, origin xyz=0.058 0.0245 0.0 rpy=0 0 0, axis -0.0 1.0 0.0
- added joint j_hfe_FR: type continuous, parent b_hfe_motor_FR, child b_kfe_motor_FR, origin xyz=0.058 -0.0245 0.0 rpy=0 0 0, axis 0.0 1.0 0.0
- added joint j_hfe_RL: type continuous, parent b_hfe_motor_RL, child b_kfe_motor_RL, origin xyz=-0.058 0.0245 -0.0 rpy=0 0 0, axis -0.0 -1.0 0.0
- added joint j_hfe_RR: type continuous, parent b_hfe_motor_RR, child b_kfe_motor_RR, origin xyz=-0.058 -0.0245 -0.0 rpy=0 0 0, axis 0.0 -1.0 -0.0
- added joint j_hfe_to_upper_leg_FL: type fixed, parent b_kfe_motor_FL, child b_upper_leg_FL, origin xyz=0.0 0.064 0.0 rpy=0 0 0
- added joint j_hfe_to_upper_leg_FR: type fixed, parent b_kfe_motor_FR, child b_upper_leg_FR, origin xyz=0.0 -0.064 0.0 rpy=0 0 0
- added joint j_hfe_to_upper_leg_RL: type fixed, parent b_kfe_motor_RL, child b_upper_leg_RL, origin xyz=0.0 0.064 0.0 rpy=0 0 0
- added joint j_hfe_to_upper_leg_RR: type fixed, parent b_kfe_motor_RR, child b_upper_leg_RR, origin xyz=0.0 -0.064 0.0 rpy=0 0 0
- added joint j_kfe_FL: type continuous, parent b_upper_leg_FL, child b_lower_leg_FL, origin xyz=-0.00018 -0.004 -0.25 rpy=0 0 0, axis 0.0 -1.0 0.0
- added joint j_kfe_FR: type continuous, parent b_upper_leg_FR, child b_lower_leg_FR, origin xyz=-0.00018 0.004 -0.25 rpy=0 0 0, axis -0.0 -1.0 -0.0
- added joint j_kfe_RL: type continuous, parent b_upper_leg_RL, child b_lower_leg_RL, origin xyz=-0.00018 -0.004 -0.25 rpy=0 0 0, axis -0.0 -1.0 -0.0
- added joint j_kfe_RR: type continuous, parent b_upper_leg_RR, child b_lower_leg_RR, origin xyz=-0.00018 0.004 -0.25 rpy=0 0 0, axis 0.0 -1.0 0.0
- added joint j_knee_to_foot_FL: type fixed, parent b_lower_leg_FL, child b_foot_FL, origin xyz=0.059113 0.011 0.21711 rpy=0 0 0
- added joint j_knee_to_foot_FR: type fixed, parent b_lower_leg_FR, child b_foot_FR, origin xyz=0.059113 -0.011 0.21711 rpy=0 0 0
- added joint j_knee_to_foot_RL: type fixed, parent b_lower_leg_RL, child b_foot_RL, origin xyz=0.059113 0.011 0.21711 rpy=0 0 0
- added joint j_knee_to_foot_RR: type fixed, parent b_lower_leg_RR, child b_foot_RR, origin xyz=0.059113 -0.011 0.21711 rpy=0 0 0

Commit message: Start full controller, this is broken release for now

File: resource/NomadFull/Nomad.urdf (robot description, URDF)
Before this commit: robot Nomad, 25 links, 24 joints
Joints:
- removed joint j_hfe_to_upper_leg_FL
- removed joint j_hfe_to_upper_leg_FR
- removed joint j_hfe_to_upper_leg_RL
- removed joint j_hfe_to_upper_leg_RR
- added joint j_hfe_to_shoulder_FL: type fixed, parent b_kfe_motor_FL, child b_upper_leg_FL, origin xyz=0.0 0.064 0.0 rpy=0 0 0
- added joint j_hfe_to_shoulder_FR: type fixed, parent b_kfe_motor_FR, child b_upper_leg_FR, origin xyz=0.0 -0.064 0.0 rpy=0 0 0
- added joint j_hfe_to_shoulder_RL: type fixed, parent b_kfe_motor_RL, child b_upper_leg_RL, origin xyz=0.0 0.064 0.0 rpy=0 0 0
- added joint j_hfe_to_shoulder_RR: type fixed, parent b_kfe_motor_RR, child b_upper_leg_RR, origin xyz=0.0 -0.064 0.0 rpy=0 0 0
- joint j_haa_FL: axis 1.0 0.0 0.0 -> -1.0 0.0 0.0
- joint j_haa_FR: axis 1.0 0.0 -0.0 -> -1.0 0.0 -0.0
- joint j_haa_RL: axis -1.0 -0.0 -0.0 -> 1.0 -0.0 -0.0
- joint j_haa_RR: axis -1.0 -0.0 -0.0 -> 1.0 -0.0 -0.0
- joint j_hfe_FL: axis -0.0 1.0 0.0 -> -0.0 -1.0 0.0
- joint j_hfe_RR: axis 0.0 -1.0 -0.0 -> 0.0 1.0 -0.0
- joint j_kfe_FR: axis -0.0 -1.0 -0.0 -> -0.0 1.0 -0.0
- joint j_kfe_RR: axis 0.0 -1.0 0.0 -> 0.0 1.0 0.0
